Commit message: fixed xacro load issue

File: catkin_ws/src/map_maker/urdf/house3.urdf.xacro (robot description, xacro)
@@ -4,5 +4,5 @@
 		<visual>
 			<geometry>
-				<mesh filename="file:///home/crazyflier/flyingcars/catkin_ws/src/map_maker/meshes/simplehouse3.dae"/>
+				<mesh filename="file://$(find map_maker)/meshes/simplehouse3.dae"/>
 			</geometry>
 		</visual>

File: catkin_ws/src/map_maker/urdf/house4.urdf.xacro (robot description, xacro)
@@ -4,5 +4,5 @@
 		<visual>
 			<geometry>
-				<mesh filename="file:///home/crazyflier/flyingcars/catkin_ws/src/map_maker/meshes/simplehouse4.dae"/>
+				<mesh filename="file://$(find map_maker)/meshes/simplehouse4.dae"/>
 			</geometry>
 		</visual>

File: catkin_ws/src/map_maker/urdf/house5.urdf.xacro (robot description, xacro)
@@ -4,5 +4,5 @@
 		<visual>
 			<geometry>
-				<mesh filename="file:///home/crazyflier/flyingcars/catkin_ws/src/map_maker/meshes/simplehouse5.dae"/>
+				<mesh filename="file://$(find map_maker)/meshes/simplehouse5.dae"/>
 			</geometry>
 		</visual>
